File: Atlas V.kicad_pcb (KiCad board)
At the start: 2 copper layers, 190 x 115 mm, 28 parts, among them J1 Alim PCB 6V, J2 +VBatt, J3 Connecteur alim driver 1, J4 Connecteur alim driver 2, U1 module_mpu6050, U2 NRF24L01P-Module-E01ML01DP5_B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, U3 LM1117MPX-3.3, U4 LM2596_Module

Commit message: PCB presque fini
Parts:
- removed Pinheader1: Driver 1, ISI-Connector_PinHeader_2.54mm:PinHeader_1x06_P2.54mm_Long_Vertical
- removed Pinheader2: Driver 2, ISI-Connector_PinHeader_2.54mm:PinHeader_1x06_P2.54mm_Long_Vertical
- added J6: Alim PCB 6V, ISI-Connector_JST:JST_XH_B2B-XH-AM_1x02_P2.50mm_Long_Vertical, F.Cu at (212.5, 197.0)
- added J7: Connecteur alim driver 1, ISI-Connector_JST:JST_XH_B2B-XH-AM_1x02_P2.50mm_Long_Vertical, F.Cu at (162.0, 197.0)
- added J8: CON 1x2 POLARIZED, ISI-Connector_Generic:AMASS_XT60-M_1x02_P7.20mm_Vertical, F.Cu at (262.5, 178.5)
- J1: value Alim PCB 6V -> Driver 1; footprint ISI-Connector_Wurth:691321100002 -> ISI-Connector_JST:JST_XH_B6B-XH-AM_1x06_P2.50mm_Long_Vertical
- J2: value +VBatt -> Connecteur alim driver 2
- J3: value Connecteur alim driver 1 -> Driver 2; footprint ISI-Connector_Wurth:691321100002 -> ISI-Connector_JST:JST_XH_B6B-XH-AM_1x06_P2.50mm_Long_Vertical
- J4: value Connecteur alim driver 2 -> Sortie batterie pour buck; footprint ISI-Connector_Wurth:691321100002 -> ISI-Connector_JST:JST_XH_B2B-XH-AM_1x02_P2.50mm_Long_Vertical
- moved J2 393.8 mm to (178.5, 197.0)
- moved D1 286.4 mm to (274.5, 186.5), turned to 180 degrees
- moved D2 240.9 mm to (271.5, 179.0), turned to -90 degrees
- moved R1 236.9 mm to (276.0, 179.1), turned to -90 degrees
- moved S1 234.2 mm to (281.5, 179.0), turned to 90 degrees
- moved J4 116.4 mm to (328.0, 201.5), turned to 0 degrees
- moved J3 85.0 mm to (207.0, 125.5), turned to 0 degrees
- moved J1 75.7 mm to (146.5, 126.5), turned to 0 degrees
- moved JST4 38.3 mm to (286.5, 158.5)
- moved U1 19.6 mm to (284.2, 131.0)
- moved C1 8.55 mm to (233.0, 178.0)
- moved C2 8.55 mm to (249.0, 180.0)
- moved U3 8.55 mm to (241.2, 178.8)
- moved A1 1.50 mm to (232.5, 112.8)
Connections:
- C1 pad 1: Net-(U3-VI) -> Net-(J2-Pin_1)
- J1 pad 1: Net-(U3-VI) -> /M1A1
- J1 pad 2: GND -> /M1B1
- J2 pad 1: Net-(D1-A) -> Net-(J2-Pin_1)
- J3 pad 1: Net-(U3-VI) -> /M1A2
- J3 pad 2: GND -> /M1B2
- J4 pad 1: Net-(U3-VI) -> unconnected-(J4-Pin_1-Pad1)
- J4 pad 2: GND -> unconnected-(J4-Pin_2-Pad2)
- U3 pad 3: Net-(U3-VI) -> Net-(J2-Pin_1)
- U4 pad 1: /Vin -> unconnected-(U4-Vin-Pad1)
- U4 pad 4: Net-(U3-VI) -> Net-(J2-Pin_1)
Routing:
- net /SDA: track 0.23 -> 301.9 mm, vias 0 -> 7
- net /SCL: track 0.00 -> 291.3 mm, vias 0 -> 8
- net /3GPIO1: track 0.00 -> 204.9 mm, vias 0 -> 7
- net /D1 GND: track 0.00 -> 195.5 mm, vias 0 -> 3
- net /2GPIO1: track 0.00 -> 191.9 mm, vias 0 -> 8
- net /XSHUT2: track 0.00 -> 191.5 mm, vias 0 -> 7
- net /Phase B2: track 0.00 -> 190.8 mm, vias 0 -> 6
- net /Phase A2: track 0.00 -> 190.6 mm, vias 0 -> 3
- net /CSN: track 0.00 -> 187.6 mm, vias 0 -> 2
- net /Phase B1: track 0.00 -> 185.7 mm, vias 0 -> 2
- net /D1 Vcc: track 0.00 -> 181.0 mm, vias 0 -> 4
- net /XSHUT1: track 0.00 -> 180.0 mm, vias 0 -> 2
- net /Phase A1: track 0.00 -> 179.8 mm, vias 0 -> 2
- net /1GPIO1: track 0.00 -> 178.9 mm, vias 0 -> 1
- net /XSHUT3: track 0.00 -> 176.7 mm, vias 0 -> 6
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- added copper zone on F.Cu, net +5V
- added copper zone on B.Cu, net GND
Other:
- outline, holes or cut-outs redrawn

Commit message: PCB terminé
Parts:
- J4: value Sortie batterie pour buck -> Sortie pcb vers buck
- moved U4 170.2 mm to (346.9, 186.7)
- moved J4 55.7 mm to (284.2, 167.0)
- moved JST8 12.8 mm to (262.2, 117.5)
- moved JST9 9.41 mm to (282.5, 117.5)
- moved JST1 6.08 mm to (301.5, 129.8)
Connections:
- J4 pad 1: unconnected-(J4-Pin_1-Pad1) -> /Vin
- J4 pad 2: unconnected-(J4-Pin_2-Pad2) -> GND
- U4 pad 1: unconnected-(U4-Vin-Pad1) -> /Vin
Routing:
- net GND: track 18.4 -> 46.7 mm
- net /D2 Vcc: track 80.7 -> 102.9 mm
- net /M3+: track 123.2 -> 141.7 mm
- net /Phase B3: track 116.8 -> 131.8 mm
- net /Phase A3: track 110.1 -> 124.6 mm
- net /M4+: track 140.9 -> 154.9 mm
- net /M3-: track 111.7 -> 125.3 mm
- net /M4-: track 132.8 -> 145.1 mm
- net /1GPIO1: track 178.9 -> 190.9 mm
- net /D2 GND: track 66.7 -> 78.2 mm
- net /Vin: track 136.0 -> 147.3 mm, vias 6 -> 4
- net /XSHUT1: track 180.0 -> 190.1 mm
- net /Phase B4: track 147.6 -> 156.8 mm
- net /Phase A4: track 142.3 -> 151.5 mm
- net /SCL: track 291.3 -> 296.2 mm
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
Commit message: PCB Terminé V2
Parts:
- removed U4: LM2596_Module, ISI-Modules:StepDown_LM2596_Module_Amazon
Connections:
- A1 pad 5V2: unconnected-(A1-SPI_5V-Pad5V2) -> +5V
- A1 pad GND4: unconnected-(A1-SPI_GND-PadGND4) -> GND
Routing:
- net Net-(J2-Pin_1): track 100.7 -> 151.2 mm
- net /Vout: track 26.4 -> 42.5 mm, vias 0 -> 2
- net /M1-: track 118.0 -> 130.8 mm
- net Net-(D1-K): track 9.28 -> 18.6 mm
- net GND: track 46.7 -> 55.7 mm, vias 0 -> 2
- net /SDA: track 303.2 -> 302.7 mm
- net Net-(A1-D18/TX1): vias 3 -> 5

Commit message: Quelques modifications à discuter de vive voix
Parts:
- added C3: 10µF, ISI-Capacitor:CP_EIA-6032-28_Kemet-C_Pad2.25x2.35mm_HandSolder, B.Cu at (248.2, 169.3)
- added F2: Fuse, ISI-Divers:Fuseholder_TR5_Littelfuse_No560_No460, F.Cu at (271.5, 185.0)
- added R2: 10K, ISI-Resistor:R_1206_3216Metric_Pad1.30x1.75mm_HandSolder, B.Cu at (147.8, 159.4)
- added R3: 10K, ISI-Resistor:R_1206_3216Metric_Pad1.30x1.75mm_HandSolder, B.Cu at (150.6, 159.4)
- added REF**: R_1206_3216Metric_Pad1.30x1.75mm_HandSolder, ISI-Resistor:R_1206_3216Metric_Pad1.30x1.75mm_HandSolder, F.Cu at (153.7, 153.7)
- moved D1 12.4 mm to (286.8, 184.7), turned to -90 degrees
- moved D2 2.24 mm to (271.3, 176.8)
- moved R1 1.99 mm to (276.1, 177.1)
Connections:
- A1 pad 5V3: unconnected-(A1-5V-Pad5V3) -> +5V
- A1 pad 5V4: unconnected-(A1-5V-Pad5V4) -> +5V
- J1 pad 4: /D1 GND -> GND
- J3 pad 4: /D2 GND -> GND
- J8 pad 1: Net-(D1-A) -> Net-(F2-Pad1)
- JST6 pad 2: /D1 GND -> GND
- JST7 pad 2: /D1 GND -> GND
- JST8 pad 2: /D2 GND -> GND
- JST9 pad 2: /D2 GND -> GND
Routing:
- net GND: track 55.7 -> 300.4 mm, vias 2 -> 7
- net /D1 GND: track 199.2 -> 0.00 mm, vias 5 -> 0
- net /D2 GND: track 78.2 -> 0.00 mm
- net +5V: track 0.00 -> 30.9 mm, vias 0 -> 2
- net Net-(F2-Pad1): track 0.00 -> 12.0 mm
- net Net-(D1-K): track 18.6 -> 7.22 mm
- net /XSHUT2: track 191.6 -> 202.8 mm
- net /XSHUT3: track 178.1 -> 182.5 mm
- net /Vout: track 42.5 -> 46.3 mm
- net /SDA: track 302.7 -> 306.2 mm
- net /SCL: track 296.2 -> 299.6 mm
- net /XSHUT1: track 190.1 -> 192.2 mm
- net Net-(D1-A): track 12.3 -> 11.1 mm
- net /1GPIO1: track 190.9 -> 190.4 mm
