File: Atlas V.kicad_sch (KiCad schematic)
At the start: 28 parts, among them J1 Alim PCB 6V, J2 +VBatt, J3 Connecteur alim driver 1, J4 Connecteur alim driver 2, U1 module_mpu6050, U2 NRF24L01P-Module-E01ML01DP5_B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, U3 LM1117MPX-3.3, U4 LM2596_Module

Commit message: Add files via upload
Parts:
- removed J1: Alim PCB 6V, ISI-Connector_Wurth:691321100002, symbol ISI-Connector_Wurth:691321100002
- removed J3: Connecteur alim driver 1, ISI-Connector_Wurth:691321100002, symbol ISI-Connector_Wurth:691321100002
- removed J4: Connecteur alim driver 2, ISI-Connector_Wurth:691321100002, symbol ISI-Connector_Wurth:691321100002
- removed Pinheader1: Driver 1, ISI-Connector_PinHeader_2.54mm:PinHeader_1x06_P2.54mm_Long_Vertical, symbol ISI-Connector_PinHeader_2.54mm:Conn_01x06_Pin
- removed Pinheader2: Driver 2, ISI-Connector_PinHeader_2.54mm:PinHeader_1x06_P2.54mm_Long_Vertical, symbol ISI-Connector_PinHeader_2.54mm:Conn_01x06_Pin
- added J1: Driver 1, ISI-Connector_JST:JST_XH_B6B-XH-AM_1x06_P2.50mm_Long_Vertical, symbol ISI-Connector_JST:Conn_01x06_Pin
- added J3: Driver 2, ISI-Connector_JST:JST_XH_B6B-XH-AM_1x06_P2.50mm_Long_Vertical, symbol ISI-Connector_JST:Conn_01x06_Pin
- added J4: Sortie batterie pour buck, ISI-Connector_JST:JST_XH_B2B-XH-AM_1x02_P2.50mm_Long_Vertical, symbol ISI-Connector_JST:Conn_01x02_Pin
- added J6: Alim PCB 6V, ISI-Connector_JST:JST_XH_B2B-XH-AM_1x02_P2.50mm_Long_Vertical, symbol ISI-Connector_JST:Conn_01x02_Pin
- added J7: Connecteur alim driver 1, ISI-Connector_JST:JST_XH_B2B-XH-AM_1x02_P2.50mm_Long_Vertical, symbol ISI-Connector_JST:Conn_01x02_Pin
- added J8: CON 1x2 POLARIZED, ISI-Connector_Generic:AMASS_XT60-M_1x02_P7.20mm_Vertical, symbol ISI-Connector_Generic:XT60_M
- J2: value +VBatt -> Connecteur alim driver 2
Connections:
- net D1 GND: now also J1.4 (Pin_4)
- net D1 Vcc: now also J1.3 (Pin_3)
- net D2 GND: now also J3.4 (Pin_4)
- net D2 Vcc: now also J3.3 (Pin_3)
- net GND: now also J6.2 (Pin_2), J7.2 (Pin_2), J8.2
- net M1A1: now also J1.1 (Pin_1)
- net M1A2: now also J3.1 (Pin_1)
- net M1B1: now also J1.2 (Pin_2)
- net M1B2: now also J3.2 (Pin_2)
- net M2A1: now also J1.5 (Pin_5)
- net M2A2: now also J3.5 (Pin_5)
- net M2B1: now also J1.6 (Pin_6)
- net M2B2: now also J3.6 (Pin_6)
- net Vin: no longer U4.1 (Vin)
- net at D1.2 (A): now also J8.1; no longer J2.1 (Pin_1)
- net at C1.1, U3.3 (VI), U4.4 (Vout): now also J2.1 (Pin_1), J6.1 (Pin_1), J7.1 (Pin_1)
Other:
- note added: "+VBatt"

Commit message: PCB terminé
Parts:
- J4: value Sortie batterie pour buck -> Sortie pcb vers buck
Connections:
- net GND: now also J4.2 (Pin_2)
- net Vin: now also J4.1 (Pin_1), U4.1 (Vin)
Changed lines of the file:
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@@
+	(wire
+		(pts
+			(xy 62.23 22.86) (xy 77.47 22.86)
+		)
+		(stroke
+			(width 0)
+			(type default)
+		)
+	)
 	(wire
 		(pts
@@
 		)
 	)
-	(label "Vin"
-		(at 67.31 22.86 0)
-		(effects
-			(font
-				(size 1.27 1.27)
-			)
-			(justify left bottom)
-		)
-	)
 	(label "XSHUT2"
 		(at 299.72 132.08 0)
@@
 			)
 			(justify right bottom)
+		)
+	)
+	(label "Vin"
+		(at 68.58 22.86 0)
+		(effects
+			(font
+				(size 1.27 1.27)
+			)
+			(justify left bottom)
 		)
 	)
@@
 	(symbol
 		(lib_id "power:GND")
+		(at 62.23 25.4 90)
+		(unit 1)
+		(exclude_from_sim no)
+		(in_bom yes)
+		(on_board yes)
+		(dnp no)
+		(fields_autoplaced yes)
+		(property "Reference" "#PWR024"
+			(at 68.58 25.4 0)
+			(effects
+				(font
+					(size 1.27 1.27)
+				)
+				(hide yes)
+			)
+		)
+		(property "Value" "GND"
+			(at 66.04 25.3999 90)
+			(effects
+				(font
+					(size 1.27 1.27)
+				)
+				(justify right)
+			)
+		)
+		(property "Footprint" ""
+			(at 62.23 25.4 0)
+			(effects
+				(font
+					(size 1.27 1.27)
+				)
+				(hide yes)
+			)
+		)
+		(property "Datasheet" ""
+			(at 62.23 25.4 0)
+			(effects
+				(font
+					(size 1.27 1.27)
+				)
+				(hide yes)
+			)
+		)
+		(property "Description" "Power symbol creates a global label with name \"GND\" , ground"
+			(at 62.23 25.4 0)
+			(effects
+				(font
+					(size 1.27 1.27)
+				)
+				(hide yes)
+			)
+		)
+		(pin "1"
+		)
+		(instances
+			(project "Atlas V"
+				(path "/ce8fccda-df24-434a-95b7-65e08a15d0db"
+					(reference "#PWR024")
+					(unit 1)
+				)
+			)
+		)
+	)
+	(symbol
+		(lib_id "power:GND")
 		(at 85.09 33.02 0)
 		(unit 1)
@@
 			)
 		)
-		(property "Value" "Sortie batterie pour buck"
+		(property "Value" "Sortie pcb vers buck"
 			(at 57.785 20.32 0)
 			(effects

Commit message: PCB Terminé V2
Connections:
- net +5V: now also A1.5V2 (SPI_5V)
- net GND: now also A1.GND4 (SPI_GND)
- no-connect marks 53 -> 51
Changed lines of the file:
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@@
 	)
 	(no_connect
-		(at 200.66 85.09)
-	)
-	(no_connect
 		(at 227.33 175.26)
 	)
@@
 	)
 	(no_connect
-		(at 198.12 85.09)
-	)
-	(no_connect
 		(at 227.33 172.72)
 	)
@@
 	(wire
 		(pts
+			(xy 203.2 81.28) (xy 203.2 85.09)
+		)
+		(stroke
+			(width 0)
+			(type default)
+		)
+	)
+	(wire
+		(pts
 			(xy 190.5 45.72) (xy 190.5 85.09)
 		)
@@
 	(wire
 		(pts
+			(xy 198.12 82.55) (xy 198.12 85.09)
+		)
+		(stroke
+			(width 0)
+			(type default)
+		)
+	)
+	(wire
+		(pts
 			(xy 261.62 93.98) (xy 269.24 93.98)
 		)
@@
 	(wire
 		(pts
+			(xy 203.2 85.09) (xy 200.66 85.09)
+		)
+		(stroke
+			(width 0)
+			(type default)
+		)
+	)
+	(wire
+		(pts
 			(xy 204.47 50.8) (xy 193.04 50.8)
 		)
@@
 	)
 	(symbol
+		(lib_id "power:GND")
+		(at 203.2 81.28 0)
+		(mirror x)
+		(unit 1)
+		(exclude_from_sim no)
+		(in_bom yes)
+		(on_board yes)
+		(dnp no)
+		(property "Reference" "#PWR026"
+			(at 203.2 74.93 0)
+			(effects
+				(font
+					(size 1.27 1.27)
+				)
+				(hide yes)
+			)
+		)
+		(property "Value" "GND"
+			(at 203.2 76.2 0)
+			(effects
+				(font
+					(size 1.27 1.27)
+				)
+			)
+		)
+		(property "Footprint" ""
+			(at 203.2 81.28 0)
+			(effects
+				(font
+					(size 1.27 1.27)
+				)
+				(hide yes)
+			)
+		)
+		(property "Datasheet" ""
+			(at 203.2 81.28 0)
+			(effects
+				(font
+					(size 1.27 1.27)
+				)
+				(hide yes)
+			)
+		)
+		(property "Description" "Power symbol creates a global label with name \"GND\" , ground"
+			(at 203.2 81.28 0)
+			(effects
+				(font
+					(size 1.27 1.27)
+				)
+				(hide yes)
+			)
+		)
+		(pin "1"
+		)
+		(instances
+			(project "Atlas V"
+				(path "/ce8fccda-df24-434a-95b7-65e08a15d0db"
+					(reference "#PWR026")
+					(unit 1)
+				)
+			)
+		)
+	)
+	(symbol
 		(lib_id "ISI-Connector_JST:Conn_01x06_Pin")
 		(at 311.15 127 0)
@@
 					(unit 1)
 				)
+			)
+		)
+	)
+	(symbol
+		(lib_id "power:+5V")
+		(at 198.12 82.55 0)
+		(unit 1)
+		(exclude_from_sim no)
+		(in_bom yes)
+		(on_board yes)
+		(dnp no)
+		(fields_autoplaced yes)
+		(property "Reference" "#PWR025"
+			(at 198.12 86.36 0)
+			(effects
+				(font
+					(size 1.27 1.27)
+				)
+				(hide yes)
+			)
+		)
+		(property "Value" "+5V"
+			(at 198.12 77.47 0)
+			(effects
+				(font
+					(size 1.27 1.27)
+				)
+			)
+		)
+		(property "Footprint" ""
+			(at 198.12 82.55 0)
+			(effects
+				(font
+					(size 1.27 1.27)
+				)
+				(hide yes)
+			)
+		)
+		(property "Datasheet" ""
+			(at 198.12 82.55 0)
+			(effects
+				(font
+					(size 1.27 1.27)
+				)
+				(hide yes)
+			)
+		)
+		(property "Description" "Power symbol creates a global label with name \"+5V\""
+			(at 198.12 82.55 0)
+			(effects
+				(font
+					(size 1.27 1.27)
+				)
+				(hide yes)
+			)
+		)
+		(pin "1"
+		)
+		(instances
+			(project "Atlas V"
+				(path "/ce8fccda-df24-434a-95b7-65e08a15d0db"
+					(reference "#PWR025")
+					(unit 1)
+				)

Commit message: Quelques modifications à discuter de vive voix
Parts:
- added C3: 10µF, ISI-Capacitor:CP_EIA-6032-28_Kemet-C_Pad2.25x2.35mm_HandSolder, symbol ISI-Capacitor:C_Polarized
- added F2: Fuse, ISI-Divers:Fuseholder_TR5_Littelfuse_No560_No460, symbol ISI-Divers:Fuse
- added R2, R3: 10K, ISI-Resistor:R_1206_3216Metric_Pad1.30x1.75mm_HandSolder, symbol ISI-Resistor:R_US_1206
Connections:
- net D1 GND is gone; now on net GND: J1.4 (Pin_4), JST6.2 (Pin_2), JST7.2 (Pin_2)
- net D2 GND is gone; now on net GND: J3.4 (Pin_4), JST8.2 (Pin_2), JST9.2 (Pin_2)
- net +5V: now also A1.5V3 (5V), A1.5V4 (5V), R2.1, R3.1
- net GND: now also C3.2
- net SCL: now also R2.2
- net SDA: now also R3.2
- net Vout: now also C3.1
- net at D1.2 (A): now also F2.2; no longer J8.1
- new net: F2.1, J8.1
- no-connect marks 51 -> 49
Other:
- moved on the sheet: J8
